Commit message: SIMBICON for Atlas robot

File: data/urdf/atlas/atlas_v3_no_head.urdf (robot description, URDF)
Before this commit: robot drc_skeleton, 28 links, 28 joints
Links:
- added link l_situational_awareness_camera_link, mass 0.1; visual box size=0.01 0.01 0.01
- added link l_situational_awareness_camera_optical_frame
- added link r_situational_awareness_camera_link, mass 0.1; visual box size=0.01 0.01 0.01
- added link r_situational_awareness_camera_optical_frame
- added link rear_situational_awareness_camera_link, mass 0.1; visual box size=0.01 0.01 0.01
- added link rear_situational_awareness_camera_optical_frame
- link l_clav: mass 2.369 -> 3.45
- link l_farm: mass 0.981 -> 3.388
- link l_foot: mass 1.634 -> 2.05
- link l_hand: mass 2.263 -> 2.509
- link l_larm: mass 2.148 -> 2.509
- link l_lglut: mass 0.69 -> 0.866
- link l_lleg: mass 4.367 -> 5.479
- link l_scap: mass 2.707 -> 3.012
- link l_talus: mass 0.1 -> 0.125
- link l_uarm: mass 1.881 -> 3.388
- link l_uglut: mass 0.5166 -> 0.648
- link l_uleg: mass 7.34 -> 9.209
- link ltorso: mass 1.92 -> 2.409
- link mtorso: mass 0.55 -> 0.69
- link pelvis: mass 14.2529 -> 17.882
- link r_clav: mass 2.369 -> 3.45
- link r_farm: mass 0.981 -> 3.388
- link r_foot: mass 1.634 -> 2.05
- link r_hand: mass 2.263 -> 2.509
- link r_larm: mass 2.148 -> 2.509
- link r_lglut: mass 0.69 -> 0.866
- link r_lleg: mass 4.367 -> 5.479
- link r_scap: mass 2.707 -> 3.012
- link r_talus: mass 0.1 -> 0.125
- link r_uarm: mass 1.881 -> 3.388
- link r_uglut: mass 0.5166 -> 0.648
- link r_uleg: mass 7.34 -> 9.209
- link utorso: mass 18.484 -> 52.007; geometry collision mesh filename=utorso.stl scale=1 1 1; collision mesh filename=utorso_pack.stl scale=1 1 1
Joints:
- removed joint back_lbz
- removed joint back_mby
- removed joint back_ubx
- removed joint l_arm_mwx
- removed joint l_arm_usy
- removed joint l_arm_uwy
- removed joint l_leg_lax
- removed joint l_leg_lhy
- removed joint l_leg_mhx
- removed joint l_leg_uay
- removed joint l_leg_uhz
- removed joint neck_ay
- removed joint r_arm_mwx
- removed joint r_arm_usy
- removed joint r_arm_uwy
- removed joint r_leg_lax
- removed joint r_leg_lhy
- removed joint r_leg_mhx
- removed joint r_leg_uay
- removed joint r_leg_uhz
- added joint back_bkx: type revolute, parent mtorso, child utorso, origin xyz=0 0 0.05 rpy=0 -0 0, axis 1 0 0, limit lower=-0.698132 upper=0.698132 effort=200 velocity=12
- added joint back_bky: type revolute, parent ltorso, child mtorso, origin xyz=0 0 0.16197 rpy=0 -0 0, axis 0 1 0, limit lower=-0.610691 upper=0.438427 effort=206.843 velocity=12
- added joint back_bkz: type revolute, parent pelvis, child ltorso, origin xyz=-0.0125 0 0 rpy=0 -0 0, axis 0 0 1, limit lower=-0.663225 upper=0.663225 effort=124.016 velocity=12
- added joint l_arm_shy: type revolute, parent utorso, child l_clav, origin xyz=0.06441 0.13866 0.10718 rpy=0 -0 0, axis 0 0.5 0.866025, limit lower=-1.5708 upper=0.785398 effort=212 velocity=12
- added joint l_arm_wrx: type revolute, parent l_farm, child l_hand, origin xyz=0 0.119 0.00921 rpy=0 -0 0, axis 1 0 0, limit lower=-1.1781 upper=1.1781 effort=60 velocity=12
- added joint l_arm_wry: type revolute, parent l_larm, child l_farm, origin xyz=0 0.187 -0.00921 rpy=0 -0 0, axis 0 1 0, limit lower=0 upper=3.14159 effort=114 velocity=12
- added joint l_leg_akx: type revolute, parent l_talus, child l_foot, origin xyz=0 0 0 rpy=0 -0 0, axis 1 0 0, limit lower=-0.8 upper=0.8 effort=90 velocity=12
- added joint l_leg_aky: type revolute, parent l_lleg, child l_talus, origin xyz=0 0 -0.422 rpy=0 -0 0, axis 0 1 0, limit lower=-1 upper=0.7 effort=700 velocity=12
- added joint l_leg_hpx: type revolute, parent l_uglut, child l_lglut, origin xyz=0 0 0 rpy=0 -0 0, axis 1 0 0, limit lower=-0.523599 upper=0.523599 effort=180 velocity=12
- added joint l_leg_hpy: type revolute, parent l_lglut, child l_uleg, origin xyz=0.05 0 -0.05 rpy=0 -0 0, axis 0 1 0, limit lower=-1.72072 upper=0.524821 effort=260 velocity=12
- added joint l_leg_hpz: type revolute, parent pelvis, child l_uglut, origin xyz=0 0.089 0 rpy=0 -0 0, axis 0 0 1, limit lower=-0.174533 upper=1.22173 effort=110 velocity=12
- added joint l_situational_awareness_camera_joint: type fixed, parent utorso, child l_situational_awareness_camera_link, origin xyz=0.216409 0.121799 0.406759 rpy=-1.57079633 0 1.30899694
- added joint l_situational_awareness_camera_optical_frame_joint: type fixed, parent l_situational_awareness_camera_link, child l_situational_awareness_camera_optical_frame, origin xyz=0 0 0 rpy=-1.5708 0.0 -1.5708
- added joint r_arm_shy: type revolute, parent utorso, child r_clav, origin xyz=0.06441 -0.13866 0.10718 rpy=0 -0 0, axis 0 0.5 -0.866025, limit lower=-1.5708 upper=0.785398 effort=212 velocity=12
- added joint r_arm_wrx: type revolute, parent r_farm, child r_hand, origin xyz=0 -0.119 0.00921 rpy=0 -0 0, axis 1 0 0, limit lower=-1.1781 upper=1.1781 effort=60 velocity=12
- added joint r_arm_wry: type revolute, parent r_larm, child r_farm, origin xyz=0 -0.187 -0.00921 rpy=0 -0 0, axis 0 1 0, limit lower=0 upper=3.14159 effort=114 velocity=12
- added joint r_leg_akx: type revolute, parent r_talus, child r_foot, origin xyz=0 0 0 rpy=0 -0 0, axis 1 0 0, limit lower=-0.8 upper=0.8 effort=90 velocity=12
- added joint r_leg_aky: type revolute, parent r_lleg, child r_talus, origin xyz=0 0 -0.422 rpy=0 -0 0, axis 0 1 0, limit lower=-1 upper=0.7 effort=700 velocity=12
- added joint r_leg_hpx: type revolute, parent r_uglut, child r_lglut, origin xyz=0 0 0 rpy=0 -0 0, axis 1 0 0, limit lower=-0.523599 upper=0.523599 effort=180 velocity=12
- added joint r_leg_hpy: type revolute, parent r_lglut, child r_uleg, origin xyz=0.05 0 -0.05 rpy=0 -0 0, axis 0 1 0, limit lower=-1.72072 upper=0.524821 effort=260 velocity=12
- added joint r_leg_hpz: type revolute, parent pelvis, child r_uglut, origin xyz=0 -0.089 0 rpy=0 -0 0, axis 0 0 1, limit lower=-1.22173 upper=0.174533 effort=110 velocity=12
- added joint r_situational_awareness_camera_joint: type fixed, parent utorso, child r_situational_awareness_camera_link, origin xyz=0.216409 -0.121799 0.406759 rpy=1.57079633 0 -1.30899694
- added joint r_situational_awareness_camera_optical_frame_joint: type fixed, parent r_situational_awareness_camera_link, child r_situational_awareness_camera_optical_frame, origin xyz=0 0 0 rpy=-1.5708 0.0 -1.5708
- added joint rear_situational_awareness_camera_joint: type fixed, parent utorso, child rear_situational_awareness_camera_link, origin xyz=-0.0026 0.0264 0.6649 rpy=0 0 3.14159
- added joint rear_situational_awareness_camera_optical_frame_joint: type fixed, parent rear_situational_awareness_camera_link, child rear_situational_awareness_camera_optical_frame, origin xyz=0 0 0 rpy=-1.5708 0.0 -1.5708
- joint l_arm_elx: origin xyz=0 0.121 0.013 rpy=0 -0 0 -> xyz=0 0.119 0.00921 rpy=0 -0 0
- joint l_arm_ely: origin xyz=0 0.185 0 rpy=0 -0 0 -> xyz=0 0.187 0.016 rpy=0 -0 0
- joint l_arm_shx: limit lower=-1.39626 upper=1.74533 effort=170 velocity=12 -> lower=-1.5708 upper=1.5708 effort=170 velocity=12; origin xyz=0 0.075 0.036 rpy=0 -0 0 -> xyz=0 0.14035 0.19609 rpy=0 -0 0
- joint l_leg_kny: limit lower=0 upper=2.45 effort=220 velocity=12 -> lower=0 upper=2.38569 effort=220 velocity=12
- joint r_arm_elx: origin xyz=0 -0.121 0.013 rpy=0 -0 0 -> xyz=0 -0.119 0.00921 rpy=0 -0 0
- joint r_arm_ely: origin xyz=0 -0.185 0 rpy=0 -0 0 -> xyz=0 -0.187 0.016 rpy=0 -0 0
- joint r_arm_shx: limit lower=-1.74533 upper=1.39626 effort=170 velocity=12 -> lower=-1.5708 upper=1.5708 effort=170 velocity=12; origin xyz=0 -0.075 0.036 rpy=0 -0 0 -> xyz=0 -0.14035 0.19609 rpy=0 -0 0
- joint r_leg_kny: limit lower=0 upper=2.45 effort=220 velocity=12 -> lower=0 upper=2.38569 effort=220 velocity=12

File: data/urdf/atlas/ground.urdf (robot description, URDF)
Before this commit: robot ground_skeleton, 2 links, 1 joints
Links:
- link ground_link: geometry collision box size=25 0.05 25; visual box size=25 0.05 25
